File: Raidillon.kicad_pcb (KiCad board)
At the start: 4 copper layers, 20.8 x 27 mm, 28 parts, among them J1 S2B-PH-SM4-TB, J2 PH1RA-03-UA, U1 113991054, U2 LPS22HHTR, U3 LIS2HH12TR, U4 TPS259621DDAR

Commit message: Removed duplicate pullup on chip enable resistor
Parts:
- R9: value RMCF0805JT4K70 -> DNP 0805
Changed lines of the file:
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@@
 		)
 		(sheetname "Root")
-		(sheetfile "Spa-Raidillon.kicad_sch")
+		(sheetfile "Raidillon.kicad_sch")
 		(attr smd)
 		(fp_line
@@
 		)
 		(sheetname "Root")
-		(sheetfile "Spa-Raidillon.kicad_sch")
+		(sheetfile "Raidillon.kicad_sch")
 		(attr smd)
 		(fp_line
@@
 			)
 		)
-		(property "Value" "RMCF0805JT4K70"
+		(property "Value" "DNP 0805"
 			(at 0 -1.65 0)
 			(layer "B.Fab")
@@
 			)
 		)
-		(property "Description" "RES 4.7K OHM 5% 1/8W 0805"
+		(property "Description" "Res 0805 Do Not Populate"
 			(at 0 0 180)
 			(unlocked yes)
@@
 			)
 		)
-		(property "Resistance" "4.7kΩ"
+		(property "Resistance" "DNP"
 			(at 0 0 180)
 			(unlocked yes)
@@
 			)
 		)
-		(property "Tolerance" "5%"
+		(property "Tolerance" "-"
 			(at 0 0 180)
 			(unlocked yes)
@@
 		)
 		(sheetname "Root")
-		(sheetfile "Spa-Raidillon.kicad_sch")
+		(sheetfile "Raidillon.kicad_sch")
 		(attr through_hole)
 		(fp_line
@@
 		)
 		(sheetname "Root")
-		(sheetfile "Spa-Raidillon.kicad_sch")
+		(sheetfile "Raidillon.kicad_sch")
 		(attr smd)
 		(fp_line

Commit message: ordered pcb
Changed lines of the file:
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@@
 			(plot_on_all_layers_selection 0x0000000_00000000)
 			(disableapertmacros no)
-			(usegerberextensions no)
-			(usegerberattributes yes)
-			(usegerberadvancedattributes yes)
-			(creategerberjobfile yes)
+			(usegerberextensions yes)
+			(usegerberattributes no)
+			(usegerberadvancedattributes no)
+			(creategerberjobfile no)
 			(dashed_line_dash_ratio 12.000000)
 			(dashed_line_gap_ratio 3.000000)
@@
 			(plotinvisibletext no)
 			(sketchpadsonfab no)
-			(subtractmaskfromsilk no)
+			(subtractmaskfromsilk yes)
 			(outputformat 1)
 			(mirror no)
-			(drillshape 1)
+			(drillshape 0)
 			(scaleselection 1)
-			(outputdirectory "")
+			(outputdirectory "RaidillonGerber/")
 		)
 	)
@@
 		(sheetname "MCU")
 		(sheetfile "mcu.kicad_sch")
-		(attr smd)
+		(attr smd dnp)
 		(fp_line
 			(start 0.227064 -0.735)
@@
 			(pinfunction "Vdd_IO")
 			(pintype "power_in")
-			(solder_mask_margin 0.05)
 		)
 		(pad "2" smd roundrect
@@
 			(pinfunction "SCL")
 			(pintype "input")
-			(solder_mask_margin 0.05)
 		)
 		(pad "3" smd roundrect
@@
 			(pinfunction "GND")
 			(pintype "passive")
-			(solder_mask_margin 0.05)
 		)
 		(pad "4" smd roundrect
@@
 			(pinfunction "SDA")
 			(pintype "bidirectional")
-			(solder_mask_margin 0.05)
 		)
 		(pad "5" smd roundrect
@@
 			(pinfunction "SA0")
 			(pintype "input")
-			(solder_mask_margin 0.05)
 		)
 		(pad "6" smd roundrect
@@
 			(pinfunction "~{CS}")
 			(pintype "input")
-			(solder_mask_margin 0.05)
 		)
 		(pad "7" smd roundrect
@@
 			(pinfunction "INT_DRDY")
 			(pintype "output")
-			(solder_mask_margin 0.05)
 		)
 		(pad "8" smd roundrect
@@
 			(pinfunction "GND")
 			(pintype "power_in")
-			(solder_mask_margin 0.05)
 		)
 		(pad "9" smd roundrect
@@
 			(pinfunction "GND")
 			(pintype "passive")
-			(solder_mask_margin 0.05)
 		)
 		(pad "10" smd roundrect
@@
 			(pinfunction "VDD")
 			(pintype "power_in")
-			(solder_mask_margin 0.05)
 		)
 		(model "${KICAD8_3DMODEL_DIR}/Package_LGA.3dshapes/ST_HLGA-10_2.5x2.5mm_P0.6mm_LayoutBorder3x2y.wrl"
@@
 	)
 	(segment
-		(start 112.5 109.45)
-		(end 112.5 107.5)
-		(width 0.254)
-		(layer "B.Cu")
-		(net 1)
-	)
-	(segment
 		(start 106.45 110)
 		(end 105.8 110)
@@
 	)
 	(segment
-		(start 109.3 110)
-		(end 111.95 110)
+		(start 115.05 106.9)
+		(end 115.05 104.95)
 		(width 0.254)
 		(layer "B.Cu")
@@
 	)
 	(segment
-		(start 112.5 107.5)
-		(end 116.175 103.825)
-		(width 0.254)
-		(layer "B.Cu")
-		(net 1)
-	)
-	(segment
 		(start 104.842976 109.546)
 		(end 104.996976 109.7)
@@
 	)
 	(segment
+		(start 109.3 110)
+		(end 111.95 110)
+		(width 0.254)
+		(layer "B.Cu")
+		(net 1)
+	)
+	(segment
 		(start 106.75 110.3)
 		(end 106.75 109.7)
@@
 	)
 	(segment
+		(start 116.175 103.825)
+		(end 116.175 103.75)
+		(width 0.254)
+		(layer "B.Cu")
+		(net 1)
+	)
+	(segment
 		(start 108.855 111.8325)
 		(end 108.9875 111.7)
@@
 	)
 	(segment
-		(start 116.175 103.825)
-		(end 116.175 103.75)
-		(width 0.254)
-		(layer "B.Cu")
-		(net 1)
-	)
-	(segment
 		(start 106.75 110.3)
 		(end 106.45 110)
@@
 	)
 	(segment
-		(start 111.95 110)
-		(end 112.5 109.45)
-		(width 0.254)
-		(layer "B.Cu")
-		(net 1)
-	)
-	(segment
 		(start 108.855 113.925)
 		(end 108.855 111.8325)
@@
 	)
 	(segment
+		(start 111.95 110)
+		(end 115.05 106.9)
+		(width 0.254)
+		(layer "B.Cu")
+		(net 1)
+	)
+	(segment
+		(start 115.05 104.95)
+		(end 116.175 103.825)
+		(width 0.254)
+		(layer "B.Cu")
+		(net 1)
+	)
+	(segment
 		(start 109.4 109.4)
 		(end 109.8 109.8)
@@
 	)
 	(via
-		(at 111.45 108.45)
+		(at 112.675 108.2)
 		(size 0.6)
 		(drill 0.3)
