File: Raidillon.kicad_sch (KiCad schematic)
At the start: 4 parts, among them J1 S2B-PH-SM4-TB, J2 PH1RA-03-UA

Commit message: ordered pcb
Other:
- title: (none) -> Radillon
Changed lines of the file:
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@@
 	(generator_version "8.0")
 	(paper "A4")
+	(title_block
+		(title "Radillon")
+		(date "2025-01-29")
+		(rev "1")
+	)
 	(junction
 		(at 73.66 104.14)
