File: sensors.kicad_sch (KiCad schematic)
At the start: 4 parts, among them U2 LPS22HHTR, U3 LIS2HH12TR

Commit message: ordered pcb
Other:
- title: (none) -> Radillon
Changed lines of the file:
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@@
 	(generator_version "8.0")
 	(paper "A4")
+	(title_block
+		(title "Radillon")
+		(date "2025-01-29")
+		(rev "1")
+	)
 	(junction
 		(at 119.38 92.71)
